File: PCB Template.kicad_sch (KiCad schematic)
At the start: 19 parts, among them U1 keyboard_parts_TEENSY2.0

Commit message: Push Changes for 32u4
Parts:
- removed U1: keyboard_parts_TEENSY2.0, teensy:Teensy2.0, symbol TEENSY 2.0:keyboard_parts_TEENSY2.0
- added C1, C2: 22pF, Capacitor_SMD:C_0805_2012Metric, symbol Device:C_Small
- added C3: 1uF, Capacitor_SMD:C_0805_2012Metric, symbol Device:C_Small
- added C4, C5, C6: 0.1uF, Capacitor_SMD:C_0805_2012Metric, symbol Device:C_Small
- added C7: 10uF, Capacitor_SMD:C_0805_2012Metric, symbol Device:C_Small
- added J1: AVR-ISP-6, Connector_PinSocket_2.54mm:PinSocket_2x03_P2.54mm_Vertical, symbol Connector:AVR-ISP-6
- added J2: Conn_01x04_MountingPin, Connector_JST:JST_SH_SM04B-SRSS-TB_1x04-1MP_P1.00mm_Horizontal, symbol Connector_Generic_MountingPin:Conn_01x04_MountingPin
- added R1: R_Small, symbol Device:R_Small
- added R2, R3: 22, Resistor_SMD:R_0805_2012Metric, symbol Device:R_Small
- added R4: 10k, Resistor_SMD:R_0805_2012Metric, symbol Device:R_Small
- added SW1: SW_PUSH, symbol device:SW_PUSH
- added U1: ATmega32U4-AU, random-keyboard-parts:atmega32u4-mu-and-au, symbol MCU_Microchip_ATmega:ATmega32U4-AU
- added Y1: 16MHz, Crystal:Crystal_SMD_3225-4Pin_3.2x2.5mm, symbol Device:Crystal_GND24_Small
Connections:
- net COL0: now also U1.41 (PF0)
- net COL1: now also U1.40 (PF1)
- net COL2: now also U1.39 (PF4)
- net ROW0: now also U1.38 (PF5)
- net ROW1: now also U1.37 (PF6)
- net ROW2: now also U1.36 (PF7)
- new net: R2.1, U1.4 (D+)
- new net: R3.2, U1.3 (D-)
- new net: C3.1, U1.6 (UCAP)
- new net: R4.1, U1.33 (~{HWB}/PE2)
- new net: C1.2, U1.16 (XTAL2), Y1.2
- new net: C2.2, U1.17 (XTAL1), Y1.4
- new net +5V: C4.1, C5.1, C6.1, C7.1, J1.2 (VCC), J2.1 (Pin_1), R1.1, U1.14 (VCC), U1.2 (UVCC), U1.24 (AVCC), U1.34 (VCC), U1.44 (AVCC), U1.7 (VBUS)
- new net D+: J2.3 (Pin_3), R2.2
- new net D-: J2.2 (Pin_2), R3.1
- new net GND: C1.1, C2.1, C3.2, C4.2, C5.2, C6.2, C7.2, J1.6 (GND), J2.4 (Pin_4), R4.2, SW1.1, U1.15 (GND), U1.23 (GND), U1.35 (GND), U1.43 (GND), U1.5 (UGND), Y1.1, Y1.3
- new net MISO: J1.1 (MISO), U1.11 (PB3)
- new net MOSI: J1.4 (MOSI), U1.10 (PB2)
- new net RST: J1.5 (~{RST}), R1.2, SW1.2, U1.13 (~{RESET})
- new net SCK: J1.3 (SCK), U1.9 (PB1)
Other:
- moved on the sheet: D1, D2, D3, D4, D5, D6, D7, D8, D9, MX1, MX2, MX3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
