File: PCB Template.kicad_pcb (KiCad board)
At the start: 2 copper layers, 71.4 x 87.3 mm, 19 parts, among them U1 keyboard_parts_TEENSY2.0

Commit message: Push Changes for 32u4
Parts:
- added C1: 22pF, Capacitor_SMD:C_0805_2012Metric, B.Cu at (126.4, 58.5)
- added C2: 22pF, Capacitor_SMD:C_0805_2012Metric, B.Cu at (132.6, 58.5)
- added C3: 1uF, Capacitor_SMD:C_0805_2012Metric, B.Cu at (122.9, 67.7)
- added C4: 0.1uF, Capacitor_SMD:C_0805_2012Metric, B.Cu at (124.2, 58.5)
- added C5: 0.1uF, Capacitor_SMD:C_0805_2012Metric, B.Cu at (139.1, 63.0)
- added C6: 0.1uF, Capacitor_SMD:C_0805_2012Metric, B.Cu at (136.4, 75.7)
- added C7: 10uF, Capacitor_SMD:C_0805_2012Metric, B.Cu at (126.4, 75.7)
- added J1: AVR-ISP-6, Connector_PinSocket_2.54mm:PinSocket_2x03_P2.54mm_Vertical, B.Cu at (101.4, 63.5)
- added J2: Conn_01x04_MountingPin, Connector_JST:JST_SH_SM04B-SRSS-TB_1x04-1MP_P1.00mm_Horizontal, B.Cu at (109.7, 65.0)
- added R2: 22, Resistor_SMD:R_0805_2012Metric, B.Cu at (122.9, 69.9)
- added R3: 22, Resistor_SMD:R_0805_2012Metric, B.Cu at (122.9, 71.8)
- added R4: 10k, Resistor_SMD:R_0805_2012Metric, B.Cu at (139.0, 73.0)
- added REF**: Unified Daughter Board Mounting Holes, random-keyboard-parts:Unified Daughter Board Mounting Holes, F.Cu at (147.0, 60.4)
- added Y1: 16MHz, Crystal:Crystal_SMD_3225-4Pin_3.2x2.5mm, B.Cu at (129.5, 58.5)
- U1: value keyboard_parts_TEENSY2.0 -> ATmega32U4-AU; footprint teensy:Teensy2.0 -> random-keyboard-parts:atmega32u4-mu-and-au; moved to B.Cu
- moved U1 13.1 mm to (131.4, 68.0)
Connections:
- U1 pad 10: unconnected-(U1-PD3) (its old number) -> MOSI
- U1 pad 11: unconnected-(U1-PC6) (its old number) -> MISO
- U1 pad 12: ROW0 -> unconnected-(U1-PB7)
- U1 pad 13: ROW1 -> RST
- U1 pad 14: unconnected-(U1-VCC)_1 -> +5V
- U1 pad 15: unconnected-(U1-GND) -> GND
- U1 pad 16: unconnected-(U1-RST) -> Net-(U1-XTAL2)
- U1 pad 17: ROW2 -> Net-(U1-XTAL1)
- U1 pad 2: COL0 -> +5V
- U1 pad 23: unconnected-(U1-PF7) -> GND
- U1 pad 24: unconnected-(U1-PF6) -> +5V
- U1 pad 3: COL1 -> Net-(U1-D-)
- U1 pad 4: COL2 -> Net-(U1-D+)
- U1 pad 5: unconnected-(U1-PB3) -> GND
- U1 pad 6: unconnected-(U1-PB7) -> Net-(U1-UCAP)
- U1 pad 7: unconnected-(U1-PD0) (its old number) -> +5V
- U1 pad 9: unconnected-(U1-PD2) (its old number) -> SCK
Routing:
- net +5V: track 0.00 -> 109.2 mm, vias 0 -> 7
- net GND: track 0.00 -> 94.3 mm
- net RST: track 0.00 -> 40.6 mm
- net MISO: track 0.00 -> 30.9 mm
- net SCK: track 0.00 -> 28.5 mm
- net COL0: track 48.6 -> 74.6 mm
- net MOSI: track 0.00 -> 25.3 mm
- net COL2: track 85.6 -> 65.5 mm
- net D-: track 0.00 -> 15.1 mm
- net ROW2: track 141.0 -> 127.2 mm
- net Net-(U1-XTAL1): track 0.00 -> 13.4 mm
- net D+: track 0.00 -> 13.3 mm
- net COL1: track 65.2 -> 52.1 mm
- net Net-(U1-XTAL2): track 0.00 -> 8.66 mm
- net Net-(U1-D-): track 0.00 -> 5.77 mm
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
Commit message: Changes to the MU/AU
Connections:
- U1 pad 45: (no net) -> GND
Routing:
- net +5V: track 109.2 -> 120.8 mm
- net unconnected-(J2-MountPin): track 0.00 -> 5.60 mm
- net unconnected-(U1-PB7): track 4.11 -> 2.99 mm
- net Net-(U1-XTAL1): track 13.4 -> 12.3 mm
- net unconnected-(U1-PB6): track 3.54 -> 2.61 mm
